File: hardware/rev. 1/project.kicad_pcb (KiCad board)
At the start: 2 copper layers, 19 x 26.6 mm, 28 parts, among them J1 Conn_Coaxial, J2 Conn_01x10, J3 Conn_01x10_1, U1 BGA725L6, U2 B4327, U3 TESEO-LIV3F, U4 ST1S12GR

Commit message: initial commit
Parts:
- R2, R3: value 0 -> DNP
- U1: footprint lib_fp:TSNP-6_0.8x0.7mm_P0.4mm -> lib_fp:TSNP-6_0.8x0.7mm_P0.4mm_1
- turned C4 to 270 degrees
Connections:
- C4 pad 1: /VCC_F -> GND
- C4 pad 2: GND -> /V_BATT
- J2 pad 5: /VCC_F -> /V_BATT
- U3 pad 6: /VCC_F -> /V_BATT
Routing:
- net /VCC_F: track 17.1 -> 3.18 mm, vias 1 -> 0
- net /V_BATT: track 0.00 -> 14.0 mm, vias 0 -> 1
