File: hardware/rev. 1/project.kicad_pcb (KiCad board)
At the start: 2 copper layers, 19 x 26.6 mm, 28 parts, among them J1 Conn_Coaxial, J2 Conn_01x10, J3 Conn_01x10_1, U1 BGA725L6, U2 B4327, U3 TESEO-LIV3F, U4 ST1S12GR

Commit message: update components list
Parts:
- removed REF**: Corner_90x0.1, lib_fp:Corner_90x0.1
- added FID1: Corner_90x0.5, lib_fp:Corner_90x0.5, F.Cu at (153.0, 97.2)
Changed lines of the file:
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@@
   (general
     (thickness 1.6)
-    (drawings 54)
+    (drawings 53)
     (tracks 208)
     (zones 0)
@@
     (add_net "Net-(U3-Pad18)")
   )
+  (module lib_fp:Corner_90x0.5 (layer F.Cu)
+    (at 152.95372 97.2312)
+    (fp_text reference FID1 (at 0.01016 -2.05994) (layer F.SilkS) hide
+      (effects (font (size 0.7 0.7) (thickness 0.15)))
+    )
+    (fp_text value Corner_90x0.5 (at 0 1.24714) (layer F.Fab)
+      (effects (font (size 1 1) (thickness 0.15)))
+    )
+    (fp_arc (start 0 0) (end 1 0) (angle -90) (layer F.Cu) (width 0.5))
+  )
   (module lib_fp:TESEO_LIV3F_SMD (layer F.Cu)
     (at 150.64704 109.9719 90)
@@
     )
   )
-  (module lib_fp:Corner_90x0.1 (layer F.Cu)
-    (at 152.94864 97.2312 90)
-    (fp_text reference REF** (at 1.27 -1.27 90) (layer F.SilkS) hide
-      (effects (font (size 0.7 0.7) (thickness 0.15)))
-    )
-    (fp_text value Corner_90x0.1 (at 1.10998 1.92278 90) (layer F.Fab)
-      (effects (font (size 0.7 0.7) (thickness 0.15)))
-    )
-    (fp_arc (start 0 0) (end 0 1) (angle -90) (layer F.Cu) (width 0.2))
-  )
   (module Resistor_SMD:R_0402_1005Metric (layer B.Cu)
     (at 148.8313 96.92386 90)
@@
     )
   )
-  (gr_arc (start 152.92832 97.24644) (end 153.9494 97.24644) (angle -90) (layer F.Cu) (width 0.5))
   (gr_text "breakout board" (at 147.9423 99.1743 90) (layer F.SilkS)
     (effects (font (size 0.7 0.7) (thickness 0.175)) (justify left))
