File: hardware/rev. 1/_autosave-project.sch (KiCad schematic (older format))
At the start: 28 parts, among them J1 Conn_Coaxial, J2 Conn_01x10, J3 Conn_01x10_1, U1 BGA725L6, U2 B4327, U3 TESEO-LIV3F, U4 ST1S12GR

Commit message: update components list
Parts:
- L1: value 5n6 -> 5.6nH
Other:
- note added: "muRata LQW15AN5N6G80D+00-21\n\nCoilcraft 0402CS-5N6XJLU"
Changed lines of the file:
@@
 P 2500 5125
 F 0 "L1" V 2690 5125 50  0000 C CNN
-F 1 "5n6" V 2599 5125 50  0000 C CNN
+F 1 "5.6nH" V 2599 5125 50  0000 C CNN
 F 2 "Inductor_SMD:L_0402_1005Metric" H 2500 5125 50  0001 C CNN
 F 3 "~" H 2500 5125 50  0001 C CNN
@@
 	1    0    0    -1
 $EndComp
+Text Notes 1400 4300 0    50   ~ 0
+muRata LQW15AN5N6G80D+00-21\n\nCoilcraft 0402CS-5N6XJLU
 $EndSCHEMATC
